Commit message: Basic state estimator implemented - unpacks state interfaces, runs pinnochio model, and performs inverse kinematics. For now, contact is always set to True.

File: src/quadruped_urdf/urdf/QuadrupedURDF_sim.urdf.xacro (robot description, xacro)
@@ -5,15 +5,18 @@
 <robot
   name="urdf" xmlns:xacro="http://www.ros.org/wiki/xacro">
-  <xacro:property name="yaml_file" value="$(find quadruped)/config/initial_joint_positions.yaml"/>
+  <xacro:property name="yaml_file" value="$(find quadruped_urdf)/config/initial_joint_positions.yaml"/>
   <xacro:property name="init_pos_yaml" value="${xacro.load_yaml(yaml_file)}"/>
   <material name="Green">
-   <color rgba="${93/255} ${255/255} ${0/255} 1.0"/>
-   </material>
+    <color rgba="${93/255} ${255/255} ${0/255} 1.0"/>
+  </material>
   <material name="Magenta">
-   <color rgba="${148/255} ${100/255} ${182/255} 1.0"/>
-   </material>
+    <color rgba="${148/255} ${100/255} ${182/255} 1.0"/>
+  </material>
   <material name="Orange">
-   <color rgba="${189/255} ${136/255} ${104/255} 1.0"/>
-   </material>
+    <color rgba="${189/255} ${136/255} ${104/255} 1.0"/>
+  </material>
+  <material name="Black">
+    <color rgba="0.05 0.05 0.05 1.0"/>
+  </material>
   <!-- Dummy link and joint so the base link is massless -->
   <link name="dummy_link" />
@@ -34,7 +37,5 @@
         <box size="0.01 0.01 0.01"/>
       </geometry>
-      <material name="red">
-        <color rgba="1 0 0 1"/>
-      </material>
+      <material name="Black"/>
     </visual>
     <collision>
@@ -73,5 +74,5 @@
       <geometry>
         <mesh
-          filename="$(find quadruped)/urdf/meshes/Body.STL" />
+          filename="$(find quadruped_urdf)/urdf/meshes/Body.STL" />
       </geometry>
       <material name="Green"/>
@@ -83,8 +84,78 @@
       <geometry>
         <mesh
-          filename="$(find quadruped)/urdf/meshes/Body.STL" />
-      </geometry>
-    </collision>
-  </link>
+          filename="$(find quadruped_urdf)/urdf/meshes/Body.STL" />
+      </geometry>
+    </collision>
+  </link>
+  <!-- Internal Components -->
+  <link name="Jetson">
+    <inertial>
+      <origin xyz="0 0 0" rpy="0 0 0"/>
+      <mass value="0.1"/>
+      <inertia ixx="0.000016" ixy="0" ixz="0" iyy="0.000016" iyz="0" izz="0.000016"/>
+    </inertial>
+    <visual>
+      <geometry>
+        <box size="0.09 0.06 0.02"/>
+      </geometry>
+      <material name="Black"/>
+    </visual>
+    <collision>
+      <geometry>
+        <box size="0.09 0.06 0.02"/>
+      </geometry>
+    </collision>
+  </link>
+  <joint name="jetson_mount" type="fixed">
+    <parent link="Body"/>
+    <child link="Jetson"/>
+    <origin xyz="0 0.15 0" rpy="0 0 0"/>
+  </joint>
+  <link name="PDB">
+    <inertial>
+      <origin xyz="0 0 0" rpy="0 0 0"/>
+      <mass value="0.05"/>
+      <inertia ixx="0.000008" ixy="0" ixz="0" iyy="0.000008" iyz="0" izz="0.000008"/>
+    </inertial>
+    <visual>
+      <geometry>
+        <box size="0.05 0.05 0.01"/>
+      </geometry>
+      <material name="Black"/>
+    </visual>
+    <collision>
+      <geometry>
+        <box size="0.05 0.05 0.01"/>
+      </geometry>
+    </collision>
+  </link>
+  <joint name="pdb_mount" type="fixed">
+    <parent link="Body"/>
+    <child link="PDB"/>
+    <origin xyz="0 0 0" rpy="0 0 0"/>
+  </joint>
+  <link name="Battery">
+    <inertial>
+      <origin xyz="0 0 0" rpy="0 0 0"/>
+      <mass value="0.3"/>
+      <inertia ixx="0.000125" ixy="0" ixz="0" iyy="0.000125" iyz="0" izz="0.000125"/>
+    </inertial>
+    <visual>
+      <geometry>
+        <box size="0.06 0.12 0.04"/>
+      </geometry>
+      <material name="Black"/>
+    </visual>
+    <collision>
+      <geometry>
+        <box size="0.06 0.12 0.04"/>
+      </geometry>
+    </collision>
+  </link>
+  <joint name="battery_mount" type="fixed">
+    <parent link="Body"/>
+    <child link="Battery"/>
+    <origin xyz="0 -.15 0" rpy="0 0 0"/>
+  </joint>
   <link
     name="Front Right Thigh">
@@ -109,5 +180,5 @@
       <geometry>
         <mesh
-          filename="$(find quadruped)/urdf/meshes/Front Right Thigh.STL" />
+          filename="$(find quadruped_urdf)/urdf/meshes/Front Right Thigh.STL" />
       </geometry>
       <material name="Magenta"/>
@@ -119,5 +190,5 @@
       <geometry>
         <mesh
-          filename="$(find quadruped)/urdf/meshes/Front Right Thigh.STL" />
+          filename="$(find quadruped_urdf)/urdf/meshes/Front Right Thigh.STL" />
       </geometry>
     </collision>
@@ -158,5 +229,5 @@
       <geometry>
         <mesh
-          filename="$(find quadruped)/urdf/meshes/Front Right Shin.STL" />
+          filename="$(find quadruped_urdf)/urdf/meshes/Front Right Shin.STL" />
       </geometry>
       <material name="Orange"/>
@@ -168,5 +239,5 @@
       <geometry>
         <mesh
-          filename="$(find quadruped)/urdf/meshes/Front Right Shin.STL" />
+          filename="$(find quadruped_urdf)/urdf/meshes/Front Right Shin.STL" />
       </geometry>
     </collision>
@@ -185,4 +256,27 @@
       xyz="0 0 -1" />
   </joint>
+  <link name="fr_foot">
+    <inertial>
+      <origin xyz="0 0 0" rpy="0 0 0"/>
+      <mass value="0.01"/>
+      <inertia ixx="0.000001" ixy="0" ixz="0" iyy="0.000001" iyz="0" izz="0.000001"/>
+    </inertial>
+    <visual>
+      <geometry>
+        <sphere radius="0.03"/>
+      </geometry>
+      <material name="Orange"/>
+    </visual>
+    <collision>
+      <geometry>
+        <sphere radius="0.03"/>
+      </geometry>
+    </collision>
+  </link>
+  <joint name="fr_foot_joint" type="fixed">
+    <parent link="Front Right Shin"/>
+    <child link="fr_foot"/>
+    <origin xyz="0.14 -0.0075 0" rpy="0 0 0"/>
+  </joint>
   <link
     name="Front Left Thigh">
@@ -207,5 +301,5 @@
       <geometry>
         <mesh
-          filename="$(find quadruped)/urdf/meshes/Front Left Thigh.STL" />
+          filename="$(find quadruped_urdf)/urdf/meshes/Front Left Thigh.STL" />
       </geometry>
       <material name="Magenta"/>
@@ -217,5 +311,5 @@
       <geometry>
         <mesh
-          filename="$(find quadruped)/urdf/meshes/Front Left Thigh.STL" />
+          filename="$(find quadruped_urdf)/urdf/meshes/Front Left Thigh.STL" />
       </geometry>
     </collision>
@@ -256,5 +350,5 @@
       <geometry>
         <mesh
-          filename="$(find quadruped)/urdf/meshes/Front Left Shin.STL" />
+          filename="$(find quadruped_urdf)/urdf/meshes/Front Left Shin.STL" />
       </geometry>
       <material name="Orange"/>
@@ -266,5 +360,5 @@
       <geometry>
         <mesh
-          filename="$(find quadruped)/urdf/meshes/Front Left Shin.STL" />
+          filename="$(find quadruped_urdf)/urdf/meshes/Front Left Shin.STL" />
       </geometry>
     </collision>
@@ -283,4 +377,27 @@
       xyz="0 0 -1" />
   </joint>
+  <link name="fl_foot">
+    <inertial>
+      <origin xyz="0 0 0" rpy="0 0 0"/>
+      <mass value="0.01"/>
+      <inertia ixx="0.000001" ixy="0" ixz="0" iyy="0.000001" iyz="0" izz="0.000001"/>
+    </inertial>
+    <visual>
+      <geometry>
+        <sphere radius="0.03"/>
+      </geometry>
+      <material name="Orange"/>
+    </visual>
+    <collision>
+      <geometry>
+        <sphere radius="0.03"/>
+      </geometry>
+    </collision>
+  </link>
+  <joint name="fl_foot_joint" type="fixed">
+    <parent link="Front Left Shin"/>
+    <child link="fl_foot"/>
+    <origin xyz="0.14 -0.0075 0" rpy="0 0 0"/>
+  </joint>
   <link
     name="Rear Right Thigh">
@@ -305,5 +422,5 @@
       <geometry>
         <mesh
-          filename="$(find quadruped)/urdf/meshes/Rear Right Thigh.STL" />
+          filename="$(find quadruped_urdf)/urdf/meshes/Rear Right Thigh.STL" />
       </geometry>
       <material name="Magenta"/>
@@ -315,5 +432,5 @@
       <geometry>
         <mesh
-          filename="$(find quadruped)/urdf/meshes/Rear Right Thigh.STL" />
+          filename="$(find quadruped_urdf)/urdf/meshes/Rear Right Thigh.STL" />
       </geometry>
     </collision>
@@ -354,5 +471,5 @@
       <geometry>
         <mesh
-          filename="$(find quadruped)/urdf/meshes/Rear Right Shin.STL" />
+          filename="$(find quadruped_urdf)/urdf/meshes/Rear Right Shin.STL" />
       </geometry>
       <material name="Orange"/>
@@ -364,5 +481,5 @@
       <geometry>
         <mesh
-          filename="$(find quadruped)/urdf/meshes/Rear Right Shin.STL" />
+          filename="$(find quadruped_urdf)/urdf/meshes/Rear Right Shin.STL" />
       </geometry>
     </collision>
@@ -381,4 +498,27 @@
       xyz="0 0 -1" />
   </joint>
+  <link name="rr_foot">
+    <inertial>
+      <origin xyz="0 0 0" rpy="0 0 0"/>
+      <mass value="0.01"/>
+      <inertia ixx="0.000001" ixy="0" ixz="0" iyy="0.000001" iyz="0" izz="0.000001"/>
+    </inertial>
+    <visual>
+      <geometry>
+        <sphere radius="0.03"/>
+      </geometry>
+      <material name="Orange"/>
+    </visual>
+    <collision>
+      <geometry>
+        <sphere radius="0.03"/>
+      </geometry>
+    </collision>
+  </link>
+  <joint name="rr_foot_joint" type="fixed">
+    <parent link="Rear Right Shin"/>
+    <child link="rr_foot"/>
+    <origin xyz="0.14 -0.0075 0" rpy="0 0 0"/>
+  </joint>
   <link
     name="Rear Left Thigh">
@@ -403,5 +543,5 @@
       <geometry>
         <mesh
-          filename="$(find quadruped)/urdf/meshes/Rear Left Thigh.STL" />
+          filename="$(find quadruped_urdf)/urdf/meshes/Rear Left Thigh.STL" />
       </geometry>
       <material name="Magenta"/>
@@ -413,5 +553,5 @@
       <geometry>
         <mesh
-          filename="$(find quadruped)/urdf/meshes/Rear Left Thigh.STL" />
+          filename="$(find quadruped_urdf)/urdf/meshes/Rear Left Thigh.STL" />
       </geometry>
     </collision>
@@ -452,5 +592,5 @@
       <geometry>
         <mesh
-          filename="$(find quadruped)/urdf/meshes/Rear Left Shin.STL" />
+          filename="$(find quadruped_urdf)/urdf/meshes/Rear Left Shin.STL" />
       </geometry>
       <material name="Orange"/>
@@ -462,5 +602,5 @@
       <geometry>
         <mesh
-          filename="$(find quadruped)/urdf/meshes/Rear Left Shin.STL" />
+          filename="$(find quadruped_urdf)/urdf/meshes/Rear Left Shin.STL" />
       </geometry>
     </collision>
@@ -479,7 +619,30 @@
       xyz="0 0 -1" />
   </joint>
+  <link name="rl_foot">
+    <inertial>
+      <origin xyz="0 0 0" rpy="0 0 0"/>
+      <mass value="0.01"/>
+      <inertia ixx="0.000001" ixy="0" ixz="0" iyy="0.000001" iyz="0" izz="0.000001"/>
+    </inertial>
+    <visual>
+      <geometry>
+        <sphere radius="0.03"/>
+      </geometry>
+      <material name="Orange"/>
+    </visual>
+    <collision>
+      <geometry>
+        <sphere radius="0.03"/>
+      </geometry>
+    </collision>
+  </link>
+  <joint name="rl_foot_joint" type="fixed">
+    <parent link="Rear Left Shin"/>
+    <child link="rl_foot"/>
+    <origin xyz="0.14 -0.0075 0" rpy="0 0 0"/>
+  </joint>
   <gazebo>
     <plugin name="gz_ros2_control::GazeboSimROS2ControlPlugin" filename="libgz_ros2_control-system.so">
-      <parameters>$(find quadruped)/config/quadruped_controllers.yaml</parameters>
+      <parameters>$(find quadruped_mpc)/config/quadruped_controllers.yaml</parameters>
       <robot_param>robot_description</robot_param>
       <robot_param_node>robot_state_publisher</robot_param_node>

Commit message: Implemented basic state estimation. State interfaces are unpacked, pinnochio model is run, and inverse kinematics are done. For now, contact is assumed True

File: src/quadruped_urdf/urdf/QuadrupedURDF_sim.urdf.xacro (robot description, xacro)
@@ -1,756 +1,25 @@
 <?xml version="1.0" encoding="utf-8"?>
-<!-- This URDF was automatically created by SolidWorks to URDF Exporter! Originally created by Stephen Brawner (brawner@gmail.com)
-     Commit Version: 1.6.0-4-g7f85cfe  Build Version: 1.6.7995.38578
-     For more information, please see http://wiki.ros.org/sw_urdf_exporter -->
-<robot
-  name="urdf" xmlns:xacro="http://www.ros.org/wiki/xacro">
-  <xacro:property name="yaml_file" value="$(find quadruped_urdf)/config/initial_joint_positions.yaml"/>
-  <xacro:property name="init_pos_yaml" value="${xacro.load_yaml(yaml_file)}"/>
-  <material name="Green">
-    <color rgba="${93/255} ${255/255} ${0/255} 1.0"/>
-  </material>
-  <material name="Magenta">
-    <color rgba="${148/255} ${100/255} ${182/255} 1.0"/>
-  </material>
-  <material name="Orange">
-    <color rgba="${189/255} ${136/255} ${104/255} 1.0"/>
-  </material>
-  <material name="Black">
-    <color rgba="0.05 0.05 0.05 1.0"/>
-  </material>
-  <!-- Dummy link and joint so the base link is massless -->
-  <link name="dummy_link" />
-  <joint name="dummy_joint" type="fixed">
-    <parent link="dummy_link" />
-    <child link="Body" />
-  </joint>
-  <!-- IMU sensor site -->
-  <link name="imu_link">
-    <inertial>
-      <mass value="0.001"/>
-      <origin xyz="0 0 0" rpy="0 0 0"/>
-      <inertia ixx="0.000001" ixy="0" ixz="0" iyy="0.000001" iyz="0" izz="0.000001"/>
-    </inertial>
-    <visual>
-      <origin xyz="0 0 0" rpy="0 0 0"/>
-      <geometry>
-        <box size="0.01 0.01 0.01"/>
-      </geometry>
-      <material name="Black"/>
-    </visual>
-    <collision>
-      <origin xyz="0 0 0" rpy="0 0 0"/>
-      <geometry>
-        <box size="0.01 0.01 0.01"/>
-      </geometry>
-    </collision>
-  </link>
-  <joint name="imu_to_body" type="fixed">
-      <parent link="Body"/>
-      <child link="imu_link"/>
-      <origin rpy="0 0 0" xyz="0 0 0"/>
-  </joint>
-  <!-- The actual robot -->
-  <link
-    name="Body">
-    <inertial>
-      <origin
-        xyz="0.000496651842729657 -0.00191436675848661 -0.00656282405798344"
-        rpy="0 0 0" />
-      <mass
-        value="2.72713096530588" />
-      <inertia
-        ixx="0.0372164866888024"
-        ixy="1.14328115404344E-11"
-        ixz="-1.84385166067456E-08"
-        iyy="0.00367331488542633"
-        iyz="1.05547030991378E-11"
-        izz="0.0370798690687598" />
-    </inertial>
-    <visual>
-      <origin
-        xyz="0 0 0"
-        rpy="0 0 0" />
-      <geometry>
-        <mesh
-          filename="$(find quadruped_urdf)/urdf/meshes/Body.STL" />
-      </geometry>
-      <material name="Green"/>
-    </visual>
-    <collision>
-      <origin
-        xyz="0 0 0"
-        rpy="0 0 0" />
-      <geometry>
-        <mesh
-          filename="$(find quadruped_urdf)/urdf/meshes/Body.STL" />
-      </geometry>
-    </collision>
-  </link>
-  <!-- Internal Components -->
-  <link name="Jetson">
-    <inertial>
-      <origin xyz="0 0 0" rpy="0 0 0"/>
-      <mass value="0.1"/>
-      <inertia ixx="0.000016" ixy="0" ixz="0" iyy="0.000016" iyz="0" izz="0.000016"/>
-    </inertial>
-    <visual>
-      <geometry>
-        <box size="0.09 0.06 0.02"/>
-      </geometry>
-      <material name="Black"/>
-    </visual>
-    <collision>
-      <geometry>
-        <box size="0.09 0.06 0.02"/>
-      </geometry>
-    </collision>
-  </link>
-  <joint name="jetson_mount" type="fixed">
-    <parent link="Body"/>
-    <child link="Jetson"/>
-    <origin xyz="0 0.15 0" rpy="0 0 0"/>
-  </joint>
-  <link name="PDB">
-    <inertial>
-      <origin xyz="0 0 0" rpy="0 0 0"/>
-      <mass value="0.05"/>
-      <inertia ixx="0.000008" ixy="0" ixz="0" iyy="0.000008" iyz="0" izz="0.000008"/>
-    </inertial>
-    <visual>
-      <geometry>
-        <box size="0.05 0.05 0.01"/>
-      </geometry>
-      <material name="Black"/>
-    </visual>
-    <collision>
-      <geometry>
-        <box size="0.05 0.05 0.01"/>
-      </geometry>
-    </collision>
-  </link>
-  <joint name="pdb_mount" type="fixed">
-    <parent link="Body"/>
-    <child link="PDB"/>
-    <origin xyz="0 0 0" rpy="0 0 0"/>
-  </joint>
-  <link name="Battery">
-    <inertial>
-      <origin xyz="0 0 0" rpy="0 0 0"/>
-      <mass value="0.3"/>
-      <inertia ixx="0.000125" ixy="0" ixz="0" iyy="0.000125" iyz="0" izz="0.000125"/>
-    </inertial>
-    <visual>
-      <geometry>
-        <box size="0.06 0.12 0.04"/>
-      </geometry>
-      <material name="Black"/>
-    </visual>
-    <collision>
-      <geometry>
-        <box size="0.06 0.12 0.04"/>
-      </geometry>
-    </collision>
-  </link>
-  <joint name="battery_mount" type="fixed">
-    <parent link="Body"/>
-    <child link="Battery"/>
-    <origin xyz="0 -.15 0" rpy="0 0 0"/>
-  </joint>
-  <link
-    name="Front Right Thigh">
-    <inertial>
-      <origin
-        xyz="2.43741414216458E-05 -0.0142051404026353 -0.00547111407205264"
-        rpy="0 0 0" />
-      <mass
-        value="0.513489297249649" />
-      <inertia
-        ixx="0.000703443703532357"
-        ixy="5.05069776934335E-07"
-        ixz="-1.25476848652197E-07"
-        iyy="0.000379089863098612"
-        iyz="-1.02974442751939E-06"
-        izz="0.00102411507237723" />
-    </inertial>
-    <visual>
-      <origin
-        xyz="0 0 0"
-        rpy="0 0 0" />
-      <geometry>
-        <mesh
-          filename="$(find quadruped_urdf)/urdf/meshes/Front Right Thigh.STL" />
-      </geometry>
-      <material name="Magenta"/>
-    </visual>
-    <collision>
-      <origin
-        xyz="0 0 0"
-        rpy="0 0 0" />
-      <geometry>
-        <mesh
-          filename="$(find quadruped_urdf)/urdf/meshes/Front Right Thigh.STL" />
-      </geometry>
-    </collision>
-  </link>
-  <joint
-    name="fr_hip"
-    type="continuous">
-    <origin
-      xyz="-0.15605 -0.1796 0"
-      rpy="1.5708 ${init_pos_yaml['initial_joint_positions']['fr_hip']} -1.5708" />
-    <parent
-      link="Body" />
-    <child
-      link="Front Right Thigh" />
-    <axis
-      xyz="0 0 -1" />
-  </joint>
-  <link
-    name="Front Right Shin">
-    <inertial>
-      <origin
-        xyz="0.1248780823163 -0.00732497518642935 0.00017505649013605"
-        rpy="0 0 0" />
-      <mass
-        value="0.129610127102807" />
-      <inertia
-        ixx="3.51684106957956E-05"
-        ixy="8.64609723784186E-07"
-        ixz="7.49065225470579E-10"
-        iyy="4.9857666056172E-05"
-        iyz="-4.6532876481813E-11"
-        izz="5.09700357908981E-05" />
-    </inertial>
-    <visual>
-      <origin
-        xyz="0 0 0"
-        rpy="0 0 0" />
-      <geometry>
-        <mesh
-          filename="$(find quadruped_urdf)/urdf/meshes/Front Right Shin.STL" />
-      </geometry>
-      <material name="Orange"/>
-    </visual>
-    <collision>
-      <origin
-        xyz="0 0 0"
-        rpy="0 0 0" />
-      <geometry>
-        <mesh
-          filename="$(find quadruped_urdf)/urdf/meshes/Front Right Shin.STL" />
-      </geometry>
-    </collision>
-  </link>
-  <joint
-    name="fr_knee"
-    type="continuous">
-    <origin
-      xyz="0 -0.13625 0.014875"
-      rpy="0 0 ${init_pos_yaml['initial_joint_positions']['fr_knee']}" />
-    <parent
-      link="Front Right Thigh" />
-    <child
-      link="Front Right Shin" />
-    <axis
-      xyz="0 0 -1" />
-  </joint>
-  <link name="fr_foot">
-    <inertial>
-      <origin xyz="0 0 0" rpy="0 0 0"/>
-      <mass value="0.01"/>
-      <inertia ixx="0.000001" ixy="0" ixz="0" iyy="0.000001" iyz="0" izz="0.000001"/>
-    </inertial>
-    <visual>
-      <geometry>
-        <sphere radius="0.03"/>
-      </geometry>
-      <material name="Orange"/>
-    </visual>
-    <collision>
-      <geometry>
-        <sphere radius="0.03"/>
-      </geometry>
-    </collision>
-  </link>
-  <joint name="fr_foot_joint" type="fixed">
-    <parent link="Front Right Shin"/>
-    <child link="fr_foot"/>
-    <origin xyz="0.14 -0.0075 0" rpy="0 0 0"/>
-  </joint>
-  <link
-    name="Front Left Thigh">
-    <inertial>
-      <origin
-        xyz="-2.69567127114678E-06 -0.0142673340488066 0.00542295719977118"
-        rpy="0 0 0" />
-      <mass
-        value="0.513479185634994" />
-      <inertia
-        ixx="0.000703377558606604"
-        ixy="-5.92700407826434E-08"
-        ixz="-6.4102146703666E-09"
-        iyy="0.000379154000610083"
-        iyz="1.03700632804851E-06"
-        izz="0.00102411493476719" />
-    </inertial>
-    <visual>
-      <origin
-        xyz="0 0 0"
-        rpy="0 0 0" />
-      <geometry>
-        <mesh
-          filename="$(find quadruped_urdf)/urdf/meshes/Front Left Thigh.STL" />
-      </geometry>
-      <material name="Magenta"/>
-    </visual>
-    <collision>
-      <origin
-        xyz="0 0 0"
-        rpy="0 0 0" />
-      <geometry>
-        <mesh
-          filename="$(find quadruped_urdf)/urdf/meshes/Front Left Thigh.STL" />
-      </geometry>
-    </collision>
-  </link>
-  <joint
-    name="fl_hip"
-    type="continuous">
-    <origin
-      xyz="0.15605 -0.1796 0"
-      rpy="1.5708 ${init_pos_yaml['initial_joint_positions']['fl_hip']} -1.5708" />
-    <parent
-      link="Body" />
-    <child
-      link="Front Left Thigh" />
-    <axis
-      xyz="0 0 -1" />
-  </joint>
-  <link
-    name="Front Left Shin">
-    <inertial>
-      <origin
-        xyz="0.124878082316303 -0.00732497518642785 0.000177556490133124"
-        rpy="0 0 0" />
-      <mass
-        value="0.129610127102807" />
-      <inertia
-        ixx="3.51684106957956E-05"
-        ixy="8.64609723784203E-07"
-        ixz="7.49065225476954E-10"
-        iyy="4.98576660561721E-05"
-        iyz="-4.653287647839E-11"
-        izz="5.09700357908982E-05" />
-    </inertial>
-    <visual>
-      <origin
-        xyz="0 0 0"
-        rpy="0 0 0" />
-      <geometry>
-        <mesh
-          filename="$(find quadruped_urdf)/urdf/meshes/Front Left Shin.STL" />
-      </geometry>
-      <material name="Orange"/>
-    </visual>
-    <collision>
-      <origin
-        xyz="0 0 0"
-        rpy="0 0 0" />
-      <geometry>
-        <mesh
-          filename="$(find quadruped_urdf)/urdf/meshes/Front Left Shin.STL" />
-      </geometry>
-    </collision>
-  </link>
-  <joint
-    name="fl_knee"
-    type="continuous">
-    <origin
-      xyz="0 -0.136249999870001 -0.015125"
-      rpy="0 0 ${init_pos_yaml['initial_joint_positions']['fl_knee']}" />
-    <parent
-      link="Front Left Thigh" />
-    <child
-      link="Front Left Shin" />
-    <axis
-      xyz="0 0 -1" />
-  </joint>
-  <link name="fl_foot">
-    <inertial>
-      <origin xyz="0 0 0" rpy="0 0 0"/>
-      <mass value="0.01"/>
-      <inertia ixx="0.000001" ixy="0" ixz="0" iyy="0.000001" iyz="0" izz="0.000001"/>
-    </inertial>
-    <visual>
-      <geometry>
-        <sphere radius="0.03"/>
-      </geometry>
-      <material name="Orange"/>
-    </visual>
-    <collision>
-      <geometry>
-        <sphere radius="0.03"/>
-      </geometry>
-    </collision>
-  </link>
-  <joint name="fl_foot_joint" type="fixed">
-    <parent link="Front Left Shin"/>
-    <child link="fl_foot"/>
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