Commit message: Dockerfile issues worked out

File: src/quadruped_urdf/urdf/body.xacro (robot description, xacro)
@@ -14,5 +14,5 @@
           rpy="0 0 0" />
         <mass
-          value="2.72713096530588" />
+          value="10" />
         <inertia
           ixx="0.0372164866888024"

File: src/quadruped_urdf/urdf/leg.xacro (robot description, xacro)
@@ -6,5 +6,5 @@
       <inertial>
         <origin xyz="2.43741414216458E-05 -0.0142051404026353 -0.00547111407205264" rpy="0 0 0"/>
-        <mass value="0.513489297249649"/>
+        <mass value=".5"/>
         <inertia ixx="0.000703443703532357" ixy="5.05069776934335E-07" ixz="-1.25476848652197E-07"
                 iyy="0.000379089863098612" iyz="-1.02974442751939E-06" izz="0.00102411507237723"/>
@@ -33,5 +33,5 @@
       <inertial>
         <origin xyz="0.124878082316303 -0.00732497518642785 0.000177556490133124" rpy="0 0 0"/>
-        <mass value="0.129610127102807"/>
+        <mass value="0.3"/>
         <inertia ixx="3.51684106957956E-05" ixy="8.64609723784203E-07" ixz="7.49065225476954E-10"
                 iyy="4.98576660561721E-05" iyz="-4.653287647839E-11" izz="5.09700357908982E-05"/>

Commit message: Confirmed OCP solver is being loaded properly in MPC controller - state estimator is miscalculating the fr leg height for some infuriating reason

File: src/quadruped_urdf/urdf/body.xacro (robot description, xacro)
@@ -3,7 +3,7 @@
   <xacro:macro name="body">
     <!-- Dummy link and joint -->
-    <link name="dummy_link" />
-    <joint name="dummy_joint" type="fixed">
-      <parent link="dummy_link" />
+    <link name="base_link" />
+    <joint name="base_fixed" type="fixed">
+      <parent link="base_link" />
       <child link="Body" />
     </joint>

Commit message: BALANCE CONTROLLER WORKS GO STUPID GO CRAZY AAAAAAAH

File: src/quadruped_urdf/urdf/body.xacro (robot description, xacro)
@@ -93,5 +93,5 @@
       <inertial>
         <origin xyz="0 0 0" rpy="0 0 0"/>
-        <mass value="0.3"/>
+        <mass value="0.1"/>
         <inertia ixx="0.000125" ixy="0" ixz="0" iyy="0.000125" iyz="0" izz="0.000125"/>
       </inertial>

File: src/quadruped_urdf/urdf/gazebo.xacro (robot description, xacro)
@@ -7,4 +7,18 @@
       <robot_param>robot_description</robot_param>
       <robot_param_node>robot_state_publisher</robot_param_node>
+    </plugin>
+    <!-- Publish ground truth odometry and pose -->
+    <plugin
+      filename="gz-sim-odometry-publisher-system"
+      name="gz::sim::systems::OdometryPublisher">
+      <dimensions>3</dimensions>
+    </plugin>
+    <plugin
+      filename="gz-sim-pose-publisher-system"
+      name="gz::sim::systems::PosePublisher">
+      <publish_link_pose>true</publish_link_pose>
+      <publish_collision_pose>false</publish_collision_pose>
+      <publish_visual_pose>false</publish_visual_pose>
+      <publish_nested_model_pose>false</publish_nested_model_pose>
     </plugin>
     <!--self_collide>true</self_collide-->

Commit message: Backup before letting agent mode loose

File: src/quadruped_urdf/urdf/body.xacro (robot description, xacro)
@@ -7,4 +7,5 @@
       <parent link="base_link" />
       <child link="Body" />
+      <origin xyz="0 0 0" rpy="0 0 0"/>
     </joint>
     <link name="Body">
@@ -29,5 +30,5 @@
         <geometry>
           <mesh
-            filename="$(find quadruped_urdf)/urdf/meshes/Body.STL" />
+            filename="file://$(find quadruped_urdf)/urdf/meshes/Body.STL" />
         </geometry>
         <material name="Green"/>
@@ -39,5 +40,5 @@
         <geometry>
           <mesh
-            filename="$(find quadruped_urdf)/urdf/meshes/Body.STL" />
+            filename="file://$(find quadruped_urdf)/urdf/meshes/Body.STL" />
         </geometry>
       </collision>

File: src/quadruped_urdf/urdf/leg.xacro (robot description, xacro)
@@ -13,5 +13,5 @@
         <origin xyz="0 0 0" rpy="0 0 0"/>
         <geometry>
-          <mesh filename="$(find quadruped_urdf)/urdf/meshes/Thigh.STL"/>
+          <mesh filename="file://$(find quadruped_urdf)/urdf/meshes/Thigh.STL"/>
         </geometry>
         <material name="Magenta"/>
@@ -20,5 +20,5 @@
         <origin xyz="0 0 0" rpy="0 0 0"/>
         <geometry>
-          <mesh filename="$(find quadruped_urdf)/urdf/meshes/Thigh.STL"/>
+          <mesh filename="file://$(find quadruped_urdf)/urdf/meshes/Thigh.STL"/>
         </geometry>
       </collision>
@@ -40,5 +40,5 @@
         <origin xyz="0 0 0" rpy="0 0 0"/>
         <geometry>
-          <mesh filename="$(find quadruped_urdf)/urdf/meshes/Shin.STL"/>
+          <mesh filename="file://$(find quadruped_urdf)/urdf/meshes/Shin.STL"/>
         </geometry>
         <material name="Orange"/>
@@ -47,5 +47,5 @@
         <origin xyz="0 0 0" rpy="0 0 0"/>
         <geometry>
-          <mesh filename="$(find quadruped_urdf)/urdf/meshes/Shin.STL"/>
+          <mesh filename="file://$(find quadruped_urdf)/urdf/meshes/Shin.STL"/>
         </geometry>
       </collision>
