Commit message: about to convert the can interface into a hpp

File: src/quadruped_urdf/urdf/quadruped_ros2_control.xacro (robot description, xacro)
@@ -1,23 +1,20 @@
-<robot name="quadruped">
-    <!-- Other robot elements... -->
-    <ros2_control name="QuadrupedHardware" type="system">
+<?xml version="1.0" encoding="utf-8"?>
+<robot name="quadruped" xmlns:xacro="http://www.ros.org/wiki/xacro">
+  <!-- ros2 plugins -->
+    <ros2_control name="quadruped_hardware" type="system">
         <hardware>
-            <plugin>quadruped_hardware/QuadrupedHardwareInterface</plugin>
+            <!-- package/class-->
+            <plugin>quadruped_hardware/ROS2CANInterface</plugin>
             <!-- CAN bus 0 configuration -->
             <param name="can_interface" value="can0"/>
             <param name="can_ids" value="1,2,3,4"/>
-            <command_interface name="CAN"/>
-            <state_interface name="CAN"/>
+            <command_interface name="CAN0_cmd"/>
+            <state_interface name="CAN0_msg"/>
             <!-- CAN bus 1 configuration -->
             <param name="can_interface" value="can1"/>
             <param name="can_ids" value="5,6,7,8"/>
-            <command_interface name="CAN"/>
-            <state_interface name="CAN"/>
+            <command_interface name="CAN1_cmd"/>
+            <state_interface name="CAN1_msg"/>
         </hardware>
-        <joint name="joint1">
-            <state_interface name="position"/>
-            <command_interface name="position"/>
-        </joint>
-        <!-- Define other joints and interfaces -->
     </ros2_control>
 </robot>

Commit message: controller manager available with more than two motors

File: src/quadruped_urdf/urdf/quadruped_ros2_control.xacro (robot description, xacro)
@@ -38,12 +38,12 @@
 <!--  -->
     <!-- </ros2_control> -->
-    <ros2_control name="quadruped_hardware/CANMotorDriver_RR" type="system">
+<!--
+    <ros2_control name="quadruped_hardware/CANMotorDriver_FRH" type="system">
         <hardware>
             <plugin>quadruped_hardware/CANMotor</plugin>
             <param name="joint_name">fr_hip</param>
             <param name="can_bus" >can0</param>
-            <param name="can_id" >25</param>
+            <param name="can_id" >10</param>
         </hardware>
-        <!-- fr_hip Joint -->
         <joint name="fr_hip">
             <command_interface name="position"/>
@@ -59,3 +59,103 @@
         </joint>
     </ros2_control>
+    <ros2_control name="quadruped_hardware/CANMotorDriver_FRK" type="system">
+        <hardware>
+            <plugin>quadruped_hardware/CANMotor</plugin>
+            <param name="joint_name">fr_knee</param>
+            <param name="can_bus" >can0</param>
+            <param name="can_id" >11</param>
+        </hardware>
+        <joint name="fr_knee">
+            <command_interface name="position"/>
+            <command_interface name="velocity"/>
+            <command_interface name="effort"/>
+            <command_interface name="kp"/>
+            <command_interface name="kd"/>
+            <command_interface name="m_state"/>
+            <state_interface name="position"/>
+            <state_interface name="velocity"/>
+            <state_interface name="effort"/>
+            <state_interface name="m_state"/>
+        </joint>
+    </ros2_control> -->
+    <ros2_control name="quadruped_hardware/CANMotorDriver_RRH" type="system" >
+        <hardware>
+            <plugin>quadruped_hardware/CANMotor</plugin>
+            <param name="joint_name">rr_hip</param>
+            <param name="can_bus" >can0</param>
+            <param name="can_id" >12</param>
+        </hardware>
+        <joint name="rr_hip">
+            <command_interface name="position"/>
+            <command_interface name="velocity"/>
+            <command_interface name="effort"/>
+            <command_interface name="kp"/>
+            <command_interface name="kd"/>
+            <command_interface name="m_state"/>
+            <state_interface name="position"/>
+            <state_interface name="velocity"/>
+            <state_interface name="effort"/>
+            <state_interface name="m_state"/>
+        </joint>
+    </ros2_control>
+    <ros2_control name="quadruped_hardware/CANMotorDriver_RRK" type="system"  >
+        <hardware>
+            <plugin>quadruped_hardware/CANMotor</plugin>
+            <param name="joint_name">rr_knee</param>
+            <param name="can_bus" >can0</param>
+            <param name="can_id" >13</param>
+        </hardware>
+        <joint name="rr_knee">
+            <command_interface name="position"/>
+            <command_interface name="velocity"/>
+            <command_interface name="effort"/>
+            <command_interface name="kp"/>
+            <command_interface name="kd"/>
+            <command_interface name="m_state"/>
+            <state_interface name="position"/>
+            <state_interface name="velocity"/>
+            <state_interface name="effort"/>
+            <state_interface name="m_state"/>
+        </joint>
+    </ros2_control>
+    <ros2_control name="quadruped_hardware/CANMotorDriver_RLH" type="system"  >
+        <hardware>
+            <plugin>quadruped_hardware/CANMotor</plugin>
+            <param name="joint_name">rl_hip</param>
+            <param name="can_bus" >can1</param>
+            <param name="can_id" >16</param>
+        </hardware>
+        <joint name="rl_hip">
+            <command_interface name="position"/>
+            <command_interface name="velocity"/>
+            <command_interface name="effort"/>
+            <command_interface name="kp"/>
+            <command_interface name="kd"/>
+            <command_interface name="m_state"/>
+            <state_interface name="position"/>
+            <state_interface name="velocity"/>
+            <state_interface name="effort"/>
+            <state_interface name="m_state"/>
+        </joint>
+    </ros2_control>
+    <!-- <ros2_control name="quadruped_hardware/CANMotorDriver_RLK" type="system">
+        <hardware>
+            <plugin>quadruped_hardware/CANMotor</plugin>
+            <param name="joint_name">rl_knee</param>
+            <param name="can_bus" >can0</param>
+            <param name="can_id" >17</param>
+        </hardware>
+        <joint name="rl_knee">
+            <command_interface name="position"/>
+            <command_interface name="velocity"/>
+            <command_interface name="effort"/>
+            <command_interface name="kp"/>
+            <command_interface name="kd"/>
+            <command_interface name="m_state"/>
+            <state_interface name="position"/>
+            <state_interface name="velocity"/>
+            <state_interface name="effort"/>
+            <state_interface name="m_state"/>
+        </joint>
+    </ros2_control> -->
 </robot>

Commit message: Motor interfaces are implemented and zeroing controller works but not in the right directions

File: src/quadruped_urdf/urdf/quadruped_ros2_control.xacro (robot description, xacro)
@@ -1,42 +1,4 @@
 <?xml version="1.0" encoding="utf-8"?>
 <robot name="quadruped" xmlns:xacro="http://www.ros.org/wiki/xacro">
- <!-- Include all component files -->
-<!-- <xacro:include filename="$(find quadruped_urdf)/urdf/properties.xacro"/>
-<xacro:include filename="$(find quadruped_urdf)/urdf/materials.xacro"/>
-<xacro:include filename="$(find quadruped_urdf)/urdf/body.xacro"/>
-<xacro:include filename="$(find quadruped_urdf)/urdf/leg.xacro"/>
-<xacro:include filename="$(find quadruped_urdf)/urdf/sensors.xacro"/> -->
-  <!-- ros2 plugins -->
-  <!-- ros2 plugins -->
-    <!-- <ros2_control name="quadruped_hardware/ROS2CANInterface" type="system"> -->
-        <!-- <hardware> -->
-            <!-- namespace/class -->
-            <!-- <plugin>quadruped_hardware/ROS2CANInterface</plugin> -->
-            <!-- <parameter> $(find quadruped_hardware)/config/quadruped_hardware.yaml </parameter> -->
-            <!-- CAN bus 0 configuration -->
-            <!-- <param name="can_interface" >can0</param> -->
-            <!-- <param name="can_ids" >10,11,12,13</param> -->
-            <!-- <param name="test">5</param> -->
-            <!-- <command_interface name="CAN0_cmd"/> -->
-            <!-- <state_interface name="CAN0_msg"/> -->
-<!--  -->
-        <!-- </hardware> -->
-    <!-- </ros2_control> -->
-    <!-- <ros2_control name="quadruped_hardware/ROS2CANInterfaceCAN" type="system"> -->
-        <!-- <hardware> -->
-            <!-- namespace/class -->
-            <!-- <plugin>quadruped_hardware/ROS2CANInterface</plugin> -->
-            <!-- <parameter> $(find quadruped_hardware)/config/quadruped_hardware.yaml </parameter> -->
-            <!-- CAN bus 0 configuration -->
-            <!-- <param name="can_interface" >can1</param> -->
-            <!-- <param name="can_ids" >10</param> -->
-            <!-- <param name="test">5</param> -->
-            <!-- <command_interface name="CAN1_cmd"/> -->
-            <!-- <state_interface name="CAN1_msg"/> -->
-<!--  -->
-        <!-- </hardware> -->
-<!--  -->
-    <!-- </ros2_control> -->
-<!--
     <ros2_control name="quadruped_hardware/CANMotorDriver_FRH" type="system">
         <hardware>
@@ -78,5 +40,5 @@
             <state_interface name="m_state"/>
         </joint>
-    </ros2_control> -->
+    </ros2_control>
     <ros2_control name="quadruped_hardware/CANMotorDriver_RRH" type="system" >
         <hardware>
@@ -119,4 +81,44 @@
         </joint>
     </ros2_control>
+    <ros2_control name="quadruped_hardware/CANMotorDriver_FLH" type="system">
+        <hardware>
+            <plugin>quadruped_hardware/CANMotor</plugin>
+            <param name="joint_name">fl_hip</param>
+            <param name="can_bus" >can1</param>
+            <param name="can_id" >14</param>
+        </hardware>
+        <joint name="fl_hip">
+            <command_interface name="position"/>
+            <command_interface name="velocity"/>
+            <command_interface name="effort"/>
+            <command_interface name="kp"/>
+            <command_interface name="kd"/>
+            <command_interface name="m_state"/>
+            <state_interface name="position"/>
+            <state_interface name="velocity"/>
+            <state_interface name="effort"/>
+            <state_interface name="m_state"/>
+        </joint>
+    </ros2_control>
+    <ros2_control name="quadruped_hardware/CANMotorDriver_FLK" type="system">
+        <hardware>
+            <plugin>quadruped_hardware/CANMotor</plugin>
+            <param name="joint_name">fl_knee</param>
+            <param name="can_bus" >can1</param>
+            <param name="can_id" >15</param>
+        </hardware>
+        <joint name="fl_knee">
+            <command_interface name="position"/>
+            <command_interface name="velocity"/>
+            <command_interface name="effort"/>
+            <command_interface name="kp"/>
+            <command_interface name="kd"/>
+            <command_interface name="m_state"/>
+            <state_interface name="position"/>
+            <state_interface name="velocity"/>
+            <state_interface name="effort"/>
+            <state_interface name="m_state"/>
+        </joint>
+    </ros2_control>
     <ros2_control name="quadruped_hardware/CANMotorDriver_RLH" type="system"  >
         <hardware>
@@ -139,9 +141,9 @@
         </joint>
     </ros2_control>
-    <!-- <ros2_control name="quadruped_hardware/CANMotorDriver_RLK" type="system">
+    <ros2_control name="quadruped_hardware/CANMotorDriver_RLK" type="system">
         <hardware>
             <plugin>quadruped_hardware/CANMotor</plugin>
             <param name="joint_name">rl_knee</param>
-            <param name="can_bus" >can0</param>
+            <param name="can_bus" >can1</param>
             <param name="can_id" >17</param>
         </hardware>
@@ -158,4 +160,4 @@
             <state_interface name="m_state"/>
         </joint>
-    </ros2_control> -->
+    </ros2_control>
 </robot>

Commit message: recovering motor work

File: src/quadruped_urdf/urdf/quadruped_ros2_control.xacro (robot description, xacro)
@@ -7,16 +7,15 @@
     </ros2_control>  -->
     <!-- setting async true here might cause a bug later -->
-    <xacro:macro name="imu_ros2_control" params="name">
-        <ros2_control name="${name}" type="sensor">
-            <hardware>
-            <plugin>quadruped_hardware/WitImuHardwareInterface</plugin>
-            <param name="device">/dev/ttyUSB0</param>
-            <param name="baud">9600</param>
-            <param name="gravity">9.797673</param>
-            <param name="product">1</param> <!-- WT901C = 1 -->
-            <param name="frame_id">imu_link</param>
-            </hardware>
-        </ros2_control>
-    </xacro:macro>
+    <ros2_control name="imu" type="sensor">
+        <hardware>
+        <plugin>quadruped_hardware/WitImuHardwareInterface</plugin>
+        <param name="device">/dev/ttyUSB0</param>
+        <param name="baud">9600</param>
+        <param name="gravity">9.797673</param>
+        <param name="product">1</param> <!-- WT901C = 1 -->
+        <param name="frame_id">imu_link</param>
+        </hardware>
+    </ros2_control>
+<!--
     <ros2_control name="quadruped_hardware/CANMotorDriver_FRH" type="system" is_async="true">
         <hardware>
@@ -65,5 +64,5 @@
         </joint>
     </ros2_control>
-    <!-- <ros2_control name="quadruped_hardware/CANMotorDriver_RRH" type="system" >
+    <ros2_control name="quadruped_hardware/CANMotorDriver_RRH" type="system" >
         <hardware>
             <plugin>quadruped_hardware/CANMotor</plugin>
@@ -110,5 +109,5 @@
             <state_interface   name="flip"/>
         </joint>
-    </ros2_control> -->
+    </ros2_control>
     <ros2_control name="quadruped_hardware/CANMotorDriver_FLH" type="system">
         <hardware>
@@ -180,5 +179,4 @@
         </joint>
     </ros2_control>
-<!--
     <ros2_control name="quadruped_hardware/CANMotorDriver_RLK" type="system">
         <hardware>
